Commit message: added camera now change transform from mount

File: arm_module_gazebo/urdf/inc/random_camera_gazebo_macro.xacro (robot description, xacro)
@@ -3,5 +3,5 @@
   <!-- Define the Xacro macro for Gazebo components -->
   <xacro:macro name="realsense_camera_gazebo" params="prefix">
-    <xacro:include filename="$(find arm_module_ur5e_description)/urdf/inc/realsense_camera_marco.xacro"/>
+    <xacro:include filename="$(find arm_module_ur5e_description)/urdf/inc/random_camera_marco.xacro"/>
     <!-- Include the camera description -->
     <xacro:realsense_camera prefix=""/>

File: arm_module_gazebo/urdf/ur_gazebo_pillar_camera.xacro (robot description, xacro)
@@ -27,8 +27,7 @@
   <xacro:include filename="$(find ur_gazebo)/urdf/ur_macro.xacro"/>
   <xacro:include filename="$(find arm_module_ur5e_description)/urdf/inc/pillar_macro.xacro"/>
-  <!--
-    WILL NEED TO INCLUDE GAZEBO
-  -->
-  <xacro:include filename="$(find arm_module_gazebo)/urdf/inc/realsense_camera_gazebo_macro.xacro"/>
+  <!-- <xacro:include filename="$(find arm_module_gazebo)/urdf/inc/random_camera_gazebo_macro.xacro"/> -->
+  <xacro:include filename="$(find arm_module_ur5e_description)/urdf/inc/_d435.urdf.xacro" />
+  <!-- <xacro:include filename="$(find arm_module_ur5e_description)/urdf/_d435.urdf.xacro" /> -->
   <!--Declare arguments -->
   <xacro:arg name="joint_limit_params" default=""/>
@@ -62,6 +61,42 @@
   <!-- Instantiate the pillar -->
   <xacro:pillar/>
+  <!-- Define the camera mount link -->
+  <link name="camera_mount">
+    <!-- Visual Representation -->
+    <visual>
+      <geometry>
+        <!-- Use the mesh for visual representation, scaled down 1000 times -->
+        <mesh filename="package://arm_module_ur5e_description/meshes/d435_mount.stl" scale="0.001 0.001 0.001"/>
+      </geometry>
+      <material name="black"/>
+    </visual>
+    <!-- Collision Representation -->
+    <collision>
+      <geometry>
+        <!-- Use the same mesh for collision -->
+        <mesh filename="package://arm_module_ur5e_description/meshes/d435_mount.stl" scale="0.001 0.001 0.001"/>
+      </geometry>
+    </collision>
+    <inertial>
+      <mass value="0.1"/>
+      <origin xyz="0 0 0" rpy="0 0 0"/>
+      <inertia ixx="0.01" ixy="0" ixz="0" iyy="0.001" iyz="0" izz="0.001"/>
+    </inertial>
+  </link>
+  <!-- Joint connecting the camera mount to the tool0 of the robot -->
+  <joint name="tool0_to_camera_mount" type="fixed">
+    <parent link="tool0"/>
+    <child link="camera_mount"/>
+    <origin xyz="0 0 0.001" rpy="0 0 0"/>
+  </joint>
   <!-- Instantiate the camera -->
-  <xacro:realsense_camera_gazebo prefix=""/>
+  <xacro:arg name="use_nominal_extrinsics" default="false"/>
+  <xacro:arg name="add_plug" default="false" />
+  <xacro:arg name="use_mesh" default="true" />
+  <!-- Instantiate the D435 camera -->
+  <xacro:sensor_d435 name="camera" topics_ns="arm_module_camera" parent="camera_mount">
+    <!-- Define the origin where the camera will be attached -->
+    <origin xyz="0.0 0.0 0.0" rpy="0 0 0"/>
+  </xacro:sensor_d435>
   <!-- Attach the components together -->
   <link name="world"/>
