Commit message: generate new urdf

File: generated_from_ur_gazebo_pillar_camera.urdf (robot description, URDF)
Before this commit: robot ur5e_robot, 18 links, 17 joints
Links:
- added link camera_back_mounting_frame
- added link camera_bottom_screw_frame
- added link camera_color_frame
- added link camera_color_optical_frame
- added link camera_depth_frame
- added link camera_depth_optical_frame
- added link camera_left_ir_frame
- added link camera_left_ir_optical_frame
- added link camera_right_ir_frame
- added link camera_right_ir_optical_frame
- link camera_link: mass 0.05 -> 0.564; geometry collision box size=0.02505 0.09 0.025; visual mesh filename=package://realsense2_description/meshes/d435.dae
- link camera_mount: geometry collision mesh filename=package://arm_module_ur5e_description/meshes/d435_mount.stl scale=0.001 0.001 0.001; visual mesh filename=package://arm_module_ur5e_description/meshes/d435_mount.stl scale=0.001 0.001 0.001
Joints:
- added joint back_mounting_joint: type fixed, parent camera_back_mounting_frame, child camera_bottom_screw_frame, origin xyz=0.0105 0 -0.0125 rpy=0 0 0
- added joint camera_color_joint: type fixed, parent camera_depth_frame, child camera_color_frame, origin xyz=0 0.015 0 rpy=0 0 0
- added joint camera_color_optical_joint: type fixed, parent camera_color_frame, child camera_color_optical_frame, origin xyz=0 0 0 rpy=-1.5707963267948966 0 -1.5707963267948966
- added joint camera_depth_joint: type fixed, parent camera_link, child camera_depth_frame, origin xyz=0 0 0 rpy=0 0 0
- added joint camera_depth_optical_joint: type fixed, parent camera_depth_frame, child camera_depth_optical_frame, origin xyz=0 0 0 rpy=-1.5707963267948966 0 -1.5707963267948966
- added joint camera_left_ir_joint: type fixed, parent camera_depth_frame, child camera_left_ir_frame, origin xyz=0 0.0 0 rpy=0 0 0
- added joint camera_left_ir_optical_joint: type fixed, parent camera_left_ir_frame, child camera_left_ir_optical_frame, origin xyz=0 0 0 rpy=-1.5707963267948966 0 -1.5707963267948966
- added joint camera_link_joint: type fixed, parent camera_bottom_screw_frame, child camera_link, origin xyz=0 0.0175 0.0125 rpy=0 0 0
- added joint camera_right_ir_joint: type fixed, parent camera_depth_frame, child camera_right_ir_frame, origin xyz=0 -0.05 0 rpy=0 0 0
- added joint camera_right_ir_optical_joint: type fixed, parent camera_right_ir_frame, child camera_right_ir_optical_frame, origin xyz=0 0 0 rpy=-1.5707963267948966 0 -1.5707963267948966
- joint camera_joint: child camera_link -> camera_back_mounting_frame; origin xyz=0 0 0.05 rpy=0 0 0 -> xyz=0 -0.045 0.02 rpy=1.5707963267948966 -1.5707963267948966 0
- joint tool0_to_camera_mount: origin xyz=0 0 0.1 rpy=0 0 0 -> xyz=0 0 0.001 rpy=0 0 0
