Commit message: restructured launch files, launched in gazebo

File: arm_module_gazebo/urdf/ur_gazebo_pillar_camera.xacro (robot description, xacro)
@@ -24,5 +24,11 @@
           xacro macro (which is hosted by ur_description).
   -->
-  <xacro:include filename="$(find arm_module_gazebo)/urdf/ur_gazebo_pillar_camera_macro.xacro"/>
+  <!-- <xacro:include filename="$(find arm_module_gazebo)/urdf/ur_gazebo_pillar_camera_macro.xacro"/> -->
+  <xacro:include filename="$(find ur_gazebo)/urdf/ur_macro.xacro"/>
+  <xacro:include filename="$(find arm_module_ur5e_description)/urdf/inc/pillar_macro.xacro"/>
+  <!--
+    WILL NEED TO INCLUDE GAZEBO
+  -->
+  <xacro:include filename="$(find arm_module_ur5e_description)/urdf/inc/realsense_camera_marco.xacro"/>
   <!--Declare arguments -->
   <xacro:arg name="joint_limit_params" default=""/>
@@ -54,17 +60,20 @@
     safety_k_position="$(arg safety_k_position)"
   />
-  <!--
-    Attach the Gazebo model to Gazebo's world frame.
-    Note: if you're looking to integrate a UR into a larger scene and need
-    to add EEFs or other parts, DO NOT change this file or the 'world' link
-    here. Create a NEW xacro instead and decide whether you need to add
-    a 'world' link there.
-  -->
-  <!-- <link name="world"/>
+  <!-- Instantiate the pillar -->
+  <xacro:pillar/>
+  <!-- Instantiate the camera -->
+  <xacro:realsense_camera prefix=""/>
+  <!-- Attach the components together -->
+  <link name="world"/>
   <joint name="world_joint" type="fixed">
     <parent link="world"/>
-    <child link="pillar"/>
+    <child link="platform"/>
     <origin xyz="0 0 0" rpy="0 0 0"/>
-  </joint> -->
+  </joint>
+  <joint name="pillar_to_base_joint" type="fixed">
+          <parent link="pillar"/>
+          <child link="base_link"/>
+          <origin xyz="0 0 0.470" rpy="0 0 ${-pi/2}"/> <!-- Position at the top of the pillar -->
+  </joint>
   <link name="tool0_controller"/>
   <joint name="tool_controller_fake_joint" type="fixed">

Commit message: add mount

File: arm_module_gazebo/urdf/ur_gazebo_pillar_camera.xacro (robot description, xacro)
@@ -30,5 +30,5 @@
     WILL NEED TO INCLUDE GAZEBO
   -->
-  <xacro:include filename="$(find arm_module_ur5e_description)/urdf/inc/realsense_camera_marco.xacro"/>
+  <xacro:include filename="$(find arm_module_gazebo)/urdf/inc/realsense_camera_gazebo_macro.xacro"/>
   <!--Declare arguments -->
   <xacro:arg name="joint_limit_params" default=""/>
@@ -63,5 +63,5 @@
   <xacro:pillar/>
   <!-- Instantiate the camera -->
-  <xacro:realsense_camera prefix=""/>
+  <xacro:realsense_camera_gazebo prefix=""/>
   <!-- Attach the components together -->
   <link name="world"/>

File: arm_module_ur5e_description/urdf/inc/realsense_camera_marco.xacro (robot description, xacro)
@@ -1,17 +1,21 @@
 <?xml version="1.0"?>
 <robot xmlns:xacro="http://wiki.ros.org/xacro">
-  <!-- Define the Xacro macro -->
+  <!-- Define the Xacro macro for robot description -->
   <xacro:macro name="realsense_camera" params="prefix">
     <!-- Define the camera mount link -->
     <link name="${prefix}camera_mount">
+      <!-- Visual Representation -->
       <visual>
         <geometry>
-          <box size="0.05 0.05 0.02"/>
+          <!-- Use the mesh for visual representation, scaled down 1000 times -->
+          <mesh filename="package://arm_module_ur5e_description/meshes/d435_mount.stl" scale="0.001 0.001 0.001"/>
         </geometry>
         <material name="black"/>
       </visual>
+      <!-- Collision Representation -->
       <collision>
         <geometry>
-          <box size="0.05 0.05 0.02"/>
+          <!-- Use the same mesh for collision -->
+          <mesh filename="package://arm_module_ur5e_description/meshes/d435_mount.stl" scale="0.001 0.001 0.001"/>
         </geometry>
       </collision>
@@ -19,5 +23,5 @@
         <mass value="0.1"/>
         <origin xyz="0 0 0" rpy="0 0 0"/>
-        <inertia ixx="0.001" ixy="0" ixz="0" iyy="0.001" iyz="0" izz="0.001"/>
+        <inertia ixx="0.01" ixy="0" ixz="0" iyy="0.001" iyz="0" izz="0.001"/>
       </inertial>
     </link>
@@ -26,5 +30,5 @@
       <parent link="tool0"/>
       <child link="${prefix}camera_mount"/>
-      <origin xyz="0 0 0.1" rpy="0 0 0"/>
+      <origin xyz="0 0 0.001" rpy="0 0 0"/>
     </joint>
     <!-- Define the camera link -->
@@ -53,29 +57,4 @@
       <origin xyz="0 0 0.05" rpy="0 0 0"/>
     </joint>
-    <!-- Gazebo plugin for the camera sensor -->
-    <gazebo>
-      <sensor type="camera" name="${prefix}camera_sensor">
-        <camera>
-          <horizontal_fov>1.047</horizontal_fov>
-          <image>
-            <width>640</width>
-            <height>480</height>
-            <format>R8G8B8</format>
-          </image>
-          <clip>
-            <near>0.01</near>
-            <far>100.0</far>
-          </clip>
-        </camera>
-        <plugin name="camera_controller" filename="libgazebo_ros_camera.so">
-          <alwaysOn>true</alwaysOn>
-          <updateRate>30.0</updateRate>
-          <cameraName>camera</cameraName>
-          <imageTopicName>camera/image_raw</imageTopicName>
-          <cameraInfoTopicName>camera/camera_info</cameraInfoTopicName>
-          <frameName>${prefix}camera_link</frameName>
-        </plugin>
-      </sensor>
-    </gazebo>
   </xacro:macro>
 </robot>

Commit message: launched with camera

File: arm_module_gazebo/urdf/ur_gazebo_pillar_camera.xacro (robot description, xacro)
@@ -19,4 +19,5 @@
     connect everything by adding the appropriate joints.
   -->
+  <xacro:property name="M_PI" value="3.1415926535897931" />
   <!--
     Import main macro.
@@ -24,10 +25,7 @@
           xacro macro (which is hosted by ur_description).
   -->
-  <!-- <xacro:include filename="$(find arm_module_gazebo)/urdf/ur_gazebo_pillar_camera_macro.xacro"/> -->
   <xacro:include filename="$(find ur_gazebo)/urdf/ur_macro.xacro"/>
   <xacro:include filename="$(find arm_module_ur5e_description)/urdf/inc/pillar_macro.xacro"/>
-  <!-- <xacro:include filename="$(find arm_module_gazebo)/urdf/inc/random_camera_gazebo_macro.xacro"/> -->
   <xacro:include filename="$(find arm_module_ur5e_description)/urdf/inc/_d435.urdf.xacro" />
-  <!-- <xacro:include filename="$(find arm_module_ur5e_description)/urdf/_d435.urdf.xacro" /> -->
   <!--Declare arguments -->
   <xacro:arg name="joint_limit_params" default=""/>
@@ -96,6 +94,5 @@
   <!-- Instantiate the D435 camera -->
   <xacro:sensor_d435 name="camera" topics_ns="arm_module_camera" parent="camera_mount">
-    <!-- Define the origin where the camera will be attached -->
-    <origin xyz="0.0 0.0 0.0" rpy="0 0 0"/>
+    <origin xyz="0 -0.045 0.02" rpy="${M_PI/2} ${-M_PI/2} 0"/>
   </xacro:sensor_d435>
   <!-- Attach the components together -->

File: arm_module_ur5e_description/urdf/inc/_d435.urdf.xacro (robot description, xacro)
@@ -31,10 +31,24 @@
 	  <color rgba="0.5 0.5 0.5 1"/>
     </material>
+    <!-- Attach back of the camera to the mount -->
+    <joint name="${name}_joint" type="fixed">
+      <xacro:insert_block name="origin" />
+      <parent link="${parent}"/> <!-- camera_mount -->
+      <child link="${name}_back_mounting_frame" />
+    </joint>
+    <!-- Create a link in the middle of two back mounting holes -->
+    <link name="${name}_back_mounting_frame"/>
+    <!-- Transfrom the back mounting frame to the bottom screw -->
+    <joint name="back_mounting_joint" type="fixed">
+      <origin xyz="0.0105 0 -0.0125" rpy="0 0 0"/>
+      <parent link="${name}_back_mounting_frame"/>
+      <child link="${name}_bottom_screw_frame"/>
+    </joint>
     <!-- camera body, with origin at bottom screw mount -->
-    <joint name="${name}_joint" type="fixed">
+    <!-- <joint name="${name}_joint" type="fixed">
       <xacro:insert_block name="origin" />
       <parent link="${parent}"/>
       <child link="${name}_bottom_screw_frame" />
-    </joint>
+    </joint> -->
     <link name="${name}_bottom_screw_frame"/>
     <joint name="${name}_link_joint" type="fixed">

Commit message: IMPORTANT setup depth processing for realsense plugin

File: arm_module_gazebo/urdf/ur_gazebo_pillar_camera.xacro (robot description, xacro)
@@ -59,7 +59,27 @@
   <!-- Instantiate the pillar -->
   <xacro:pillar/>
+  <!-- Instantiate the camera -->
+  <xacro:arg name="use_nominal_extrinsics" default="false"/>
+  <xacro:arg name="add_plug" default="false" />
+  <xacro:arg name="use_mesh" default="true" />
+  <!-- Instantiate the D435 camera -->
+  <xacro:sensor_d435 name="camera" topics_ns="arm_module_camera" parent="camera_mount">
+    <origin xyz="0 -0.045 0.02" rpy="${M_PI/2} ${-M_PI/2} 0"/>
+  </xacro:sensor_d435>
+  <!-- Attach the components together -->
+  <!-- -->
+  <joint name="pillar_to_base_joint" type="fixed">
+          <parent link="pillar"/>
+          <child link="base_link"/>
+          <origin xyz="0 0 0.470" rpy="0 0 ${-pi/2}"/> <!-- Position at the top of the pillar -->
+  </joint>
+  <link name="tool0_controller"/>
+  <joint name="tool_controller_fake_joint" type="fixed">
+    <parent link="tool0"/>
+    <child link="tool0_controller"/>
+    <origin xyz="0 0 0" rpy="0 0 0"/>
+  </joint>
   <!-- Define the camera mount link -->
   <link name="camera_mount">
-    <!-- Visual Representation -->
     <visual>
       <geometry>
@@ -69,5 +89,4 @@
       <material name="black"/>
     </visual>
-    <!-- Collision Representation -->
     <collision>
       <geometry>
@@ -88,13 +107,4 @@
     <origin xyz="0 0 0.001" rpy="0 0 0"/>
   </joint>
-  <!-- Instantiate the camera -->
-  <xacro:arg name="use_nominal_extrinsics" default="false"/>
-  <xacro:arg name="add_plug" default="false" />
-  <xacro:arg name="use_mesh" default="true" />
-  <!-- Instantiate the D435 camera -->
-  <xacro:sensor_d435 name="camera" topics_ns="arm_module_camera" parent="camera_mount">
-    <origin xyz="0 -0.045 0.02" rpy="${M_PI/2} ${-M_PI/2} 0"/>
-  </xacro:sensor_d435>
-  <!-- Attach the components together -->
   <link name="world"/>
   <joint name="world_joint" type="fixed">
@@ -103,14 +113,3 @@
     <origin xyz="0 0 0" rpy="0 0 0"/>
   </joint>
-  <joint name="pillar_to_base_joint" type="fixed">
-          <parent link="pillar"/>
-          <child link="base_link"/>
-          <origin xyz="0 0 0.470" rpy="0 0 ${-pi/2}"/> <!-- Position at the top of the pillar -->
-  </joint>
-  <link name="tool0_controller"/>
-  <joint name="tool_controller_fake_joint" type="fixed">
-    <parent link="tool0"/>
-    <child link="tool0_controller"/>
-    <origin xyz="0 0 0" rpy="0 0 0"/>
-  </joint>
 </robot>
