Commit message: set initial joint positions

File: arm_module_gazebo/urdf/ur_gazebo_pillar_realsense.xacro (robot description, xacro)
@@ -87,5 +87,4 @@
         <mesh filename="package://arm_module_ur5e_description/meshes/d435_mount.stl" scale="0.001 0.001 0.001"/>
       </geometry>
-      <material name="black"/>
     </visual>
     <collision>
